File: Motor.sch (KiCad schematic (older format))
At the start: 22 parts, among them J2 Screw_Terminal_01x02, J3 Screw_Terminal_01x02, Q1 PSMN9R1-30YL, Q2 PSMN9R1-30YL, U2 IRS2008S, U3 LD1117S50TR_SOT223, U4 LTV-357T, U5 LTV-357T

Commit message: changed optocouplers
Parts:
- removed C10: C1206C106K4RACTU, Capacitor_SMD:C_1206_3216Metric_Pad1.33x1.80mm_HandSolder, symbol Device:C
- removed C9: 100n, Capacitor_SMD:C_0603_1608Metric_Pad1.08x0.95mm_HandSolder, symbol Device:C
- removed R10: 100, Resistor_SMD:R_0603_1608Metric_Pad0.98x0.95mm_HandSolder, symbol Device:R
- removed R12, R13: 4.7k, Resistor_SMD:R_0603_1608Metric_Pad0.98x0.95mm_HandSolder, symbol Device:R
- removed U3: LD1117S50TR_SOT223, Package_TO_SOT_SMD:SOT-223-3_TabPin2, symbol Regulator_Linear:LD1117S50TR_SOT223
- removed U4, U5: LTV-357T, Package_SO:SO-4_4.4x3.6mm_P2.54mm, symbol Isolator:LTV-357T
- added R?: 100, Resistor_SMD:R_0603_1608Metric_Pad0.98x0.95mm_HandSolder, symbol Device:R
- added U4, U?: H11L1, symbol Isolator:H11L1
Connections:
- net labels removed: +5P
- wire segments 77 -> 62
Other:
- moved on the sheet: R11
